File: MCPL3-AC-V.brd (EAGLE design)
At the start: 20 x 15 mm, 4 parts, among them X1 TSW-104-07-G-S

Commit message: Add files via upload
New logo update
Parts:
- moved U$2 0.90 mm to (5.80, 5.00)
Changed lines of the file:
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@@
 </element>
 <element name="LOGO1" library="SparkFun-Aesthetics" package="OSHW-LOGO-MINI" value="OSHW-LOGOMINI" x="2.5" y="1.5" smashed="yes" grouprefs="PCB"/>
-<element name="U$2" library="logo_vokolo" package="LOGO_VOKOLO_9,8MM" value="LOGO_VOKOLO12MM" x="4.9" y="5" smashed="yes"/>
+<element name="U$2" library="logo_vokolo" package="LOGO_VOKOLO_9,8MM" value="LOGO_VOKOLO12MM" x="5.8" y="5" smashed="yes"/>
 </elements>
 <signals>
