File: MCPL3-AC-V.sch (EAGLE design)
At the start: 4 parts, among them X1 TSW-104-07-G-S

Commit message: Add files via upload
New logo update
Changed lines of the file:
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@@
 </instance>
 <instance part="LOGO1" gate="G$1" x="81.28" y="48.26" smashed="yes"/>
-<instance part="U$2" gate="G$1" x="40.64" y="43.18" smashed="yes"/>
+<instance part="U$2" gate="VOKOLO" x="76.2" y="60.96" smashed="yes"/>
 </instances>
 <busses>
